Commit message: Update lite6_robot.urdf.xacro
bakjes dieper

File: src/my_xarm_lite6/urdf/lite6_robot.urdf.xacro (robot description, xacro)
@@ -87,5 +87,7 @@
                     izz="${2*m*r*r/5}" />
   </xacro:macro>
-  <link name="world" />
+  <link name="world">
+   <origin xyz="0 0 0"/>
+  </link>
   <link name="baseplate_link">
     <visual>
@@ -142,5 +144,5 @@
     <origin xyz="0.0 0.0 0.0" rpy="0.0 0.0 0.0"/>
   </joint>
-<!-- 		Muur definieren 		-->
+ //////////////////////////////////////////////////////////////////////////////////////////////////
 <link name="muur_base_link">
     <visual>
@@ -163,50 +165,82 @@
     <child link="muur_base_link" />
   </joint>
-<!-- 		Camera definieren 		-->
+//////////////////////////////////////////////////////////////////////////////////////////////////
 <link name="camera_base_link">
-        <visual>
-            <origin xyz="0.0 0.0 0.39"/>
-            <geometry>
-                <box size="0.03 0.03 0.78"/>
-            </geometry>
-            <material name="LightGrey"/>
-        </visual>
-    </link>
-    <joint name="camera_base_joint" type="fixed">
-        <origin xyz="-0.03 0.65 0.0"/>
-        <parent link="world"/>
-        <child link="camera_base_link"/>
-    </joint>
-    <link name="camera_top_link">
-        <visual>
-            <origin xyz="-0.25 0.0 0.015"/>
-            <geometry>
-                <box size="0.5 0.03 0.03"/>
-            </geometry>
-            <material name="LightGrey"/>
-        </visual>
-    </link>
-    <joint name="camera_top_link_joint" type="fixed">
-        <origin xyz="0.135 0 0.78"/>
-        <parent link="camera_base_link"/>
-        <child link="camera_top_link"/>
-    </joint>
-  <link name="camera_link">
-    <visual>
-      <origin xyz="-0.055 0.0 -0.2" />
+    <visual>
+      <origin xyz="0.0 0.0 0.39"/>
+      <geometry>
+        <box size="0.03 0.03 0.78"/>
+      </geometry>
+	<material name="LightGrey"/>
+    </visual>
+  </link>
+  <joint name="camera_base_joint" type="fixed">
+    <origin xyz="-0.03 0.65 0.0"/>
+    <parent link="world"/>
+    <child link="camera_base_link"/>
+  </joint>
+<link name="camera_top_link">
+      <visual>
+      <origin xyz="-0.25 0.0 0.015"/>
+      <geometry>
+        <box size="0.5 0.03 0.03"/>
+      </geometry>
+	<material name="LightGrey"/>
+    </visual>
+  </link>
+  <joint name="camera_top_link_joint" type="fixed">
+    <origin xyz="0.135 0 0.78"/>
+    <parent link="camera_base_link"/>
+    <child link="camera_top_link"/>
+  </joint>
+//////////////////////////////////////////////////////////////////////////////////////////////
+<link name="camera_link">
+    <visual>
+      <origin xyz="-0.055 0.0 -0.02 " />
+      <geometry>
+        <box size="0.11 0.03 0.04" />
+      </geometry>
       <material name="test"/>
     </visual>
   </link>
   <joint name="camera_joint" type="fixed">
-    <origin xyz="-0.305 0.64 0.76" rpy="1.53 1.53 3.1415" />
-    <parent link="world" />
+    <origin xyz="-0.39 0.0 0" />
+    <parent link="camera_top_link" />
     <child link="camera_link" />
   </joint>
-<!-- 		Bakken definieren		 -->
+/////////////////////////////////////////////////////////////////////////////////////////////
  <link name="Bak_een_link">
     <visual>
-      <origin xyz="0.05 -0.0875 0.035" />
-      <geometry>
-        <box size="0.1 0.175 0.07" />
+      <origin xyz="0.004 -0.0875 0.035" />
+      <geometry>
+        <box size="0.008 0.175 0.07" />
+      </geometry>
+      <material name="blue"/>
+    </visual>
+   <visual>
+      <origin xyz="0.05 -0.0875 0.0025" />
+      <geometry>
+        <box size="0.1 0.175 0.005" />
+      </geometry>
+      <material name="blue"/>
+    </visual>
+   <visual>
+      <origin xyz="0.096 -0.0875 0.035" />
+      <geometry>
+        <box size="0.008 0.175 0.07" />
+      </geometry>
+      <material name="blue"/>
+    </visual>
+   <visual>
+      <origin xyz="0.05 -0.004 0.017" />
+      <geometry>
+        <box size="0.1 0.008 0.034" />
+      </geometry>
+      <material name="blue"/>
+    </visual>
+  <visual>
+      <origin xyz="0.05 -0.1775 0.035" />
+      <geometry>
+        <box size="0.1 0.008 0.07" />
       </geometry>
       <material name="blue"/>
@@ -219,8 +253,36 @@
   </joint>
 <link name="Bak_twee_link">
-    <visual>
-      <origin xyz="0.05 -0.0875 0.035" />
-      <geometry>
-        <box size="0.1 0.175 0.07" />
+     <visual>
+      <origin xyz="0.004 -0.0875 0.035" />
+      <geometry>
+        <box size="0.008 0.175 0.07" />
+      </geometry>
+      <material name="blue"/>
+    </visual>
+   <visual>
+      <origin xyz="0.05 -0.0875 0.0025" />
+      <geometry>
+        <box size="0.1 0.175 0.005" />
+      </geometry>
+      <material name="blue"/>
+    </visual>
+   <visual>
+      <origin xyz="0.096 -0.0875 0.035" />
+      <geometry>
+        <box size="0.008 0.175 0.07" />
+      </geometry>
+      <material name="blue"/>
+    </visual>
+   <visual>
+      <origin xyz="0.05 -0.004 0.017" />
+      <geometry>
+        <box size="0.1 0.008 0.034" />
+      </geometry>
+      <material name="blue"/>
+    </visual>
+  <visual>
+      <origin xyz="0.05 -0.1775 0.035" />
+      <geometry>
+        <box size="0.1 0.008 0.07" />
       </geometry>
       <material name="blue"/>
@@ -234,12 +296,40 @@
 <link name="Bak_drie_link">
     <visual>
-      <origin xyz="0.05 -0.0875 0.035" />
-      <geometry>
-        <box size="0.1 0.175 0.07" />
-      </geometry>
-      <material name="blue"/>
-    </visual>
-  </link>
-<joint name="Bak_drie" type="fixed">
+      <origin xyz="0.004 -0.0875 0.035" />
+      <geometry>
+        <box size="0.008 0.175 0.07" />
+      </geometry>
+      <material name="blue"/>
+    </visual>
+   <visual>
+      <origin xyz="0.05 -0.0875 0.0025" />
+      <geometry>
+        <box size="0.1 0.175 0.005" />
+      </geometry>
+      <material name="blue"/>
+    </visual>
+   <visual>
+      <origin xyz="0.096 -0.0875 0.035" />
+      <geometry>
+        <box size="0.008 0.175 0.07" />
+      </geometry>
+      <material name="blue"/>
+    </visual>
+   <visual>
+      <origin xyz="0.05 -0.004 0.017" />
+      <geometry>
+        <box size="0.1 0.008 0.034" />
+      </geometry>
+      <material name="blue"/>
+    </visual>
+  <visual>
+      <origin xyz="0.05 -0.1775 0.035" />
+      <geometry>
+        <box size="0.1 0.008 0.07" />
+      </geometry>
+      <material name="blue"/>
+    </visual>
+  </link>
+ <joint name="Bak_drie" type="fixed">
     <origin xyz="-0.105 -0.055 0.07" />
     <parent link="Bak_een_link" />
@@ -248,7 +338,35 @@
 <link name="Bak_vier_link">
     <visual>
-      <origin xyz="0.05 -0.0875 0.035" />
-      <geometry>
-        <box size="0.1 0.175 0.07" />
+      <origin xyz="0.004 -0.0875 0.035" />
+      <geometry>
+        <box size="0.008 0.175 0.07" />
+      </geometry>
+      <material name="blue"/>
+    </visual>
+   <visual>
+      <origin xyz="0.05 -0.0875 0.0025" />
+      <geometry>
+        <box size="0.1 0.175 0.005" />
+      </geometry>
+      <material name="blue"/>
+    </visual>
+   <visual>
+      <origin xyz="0.096 -0.0875 0.035" />
+      <geometry>
+        <box size="0.008 0.175 0.07" />
+      </geometry>
+      <material name="blue"/>
+    </visual>
+   <visual>
+      <origin xyz="0.05 -0.004 0.017" />
+      <geometry>
+        <box size="0.1 0.008 0.034" />
+      </geometry>
+      <material name="blue"/>
+    </visual>
+  <visual>
+      <origin xyz="0.05 -0.1775 0.035" />
+      <geometry>
+        <box size="0.1 0.008 0.07" />
       </geometry>
       <material name="blue"/>
@@ -260,9 +378,9 @@
     <child link="Bak_vier_link" />
   </joint>
-<!-- 		Grippper definieren 		-->
+////////////////////////////////////////////////////////////////////
 <link name="cylinder_link">
     <visual>
       <geometry>
-        <cylinder radius="0.04" length="0.06"/>
+        <cylinder radius="0.0375" length="0.045"/>
       </geometry>
       <material name="test"/>
@@ -270,7 +388,20 @@
   </link>
 <joint name="cylinder" type="fixed">
-    <origin xyz="0.0 0.0 0.04" />
+    <origin xyz="0.0 0.0 0.0225" />
     <parent link="tcp_link" />
     <child link="cylinder_link" />
   </joint>
+<link name="gripper_link">
+    <visual>
+      <geometry>
+        <box size="0.05 0.02 0.025" />
+      </geometry>
+      <material name="test"/>
+    </visual>
+  </link>
+<joint name="gripper" type="fixed">
+    <origin xyz="0.0 0.0 0.025" />
+    <parent link="cylinder_link" />
+    <child link="gripper_link" />
+  </joint>
 </robot>

Commit message: Update lite6_robot.urdf.xacro
wijziging camera

File: src/my_xarm_lite6/urdf/lite6_robot.urdf.xacro (robot description, xacro)
@@ -166,45 +166,45 @@
   </joint>
 //////////////////////////////////////////////////////////////////////////////////////////////////
+<!-- 		Camera definieren 		-->
 <link name="camera_base_link">
-    <visual>
-      <origin xyz="0.0 0.0 0.39"/>
-      <geometry>
-        <box size="0.03 0.03 0.78"/>
-      </geometry>
-	<material name="LightGrey"/>
-    </visual>
-  </link>
-  <joint name="camera_base_joint" type="fixed">
-    <origin xyz="-0.03 0.65 0.0"/>
-    <parent link="world"/>
-    <child link="camera_base_link"/>
-  </joint>
-<link name="camera_top_link">
-      <visual>
-      <origin xyz="-0.25 0.0 0.015"/>
-      <geometry>
-        <box size="0.5 0.03 0.03"/>
-      </geometry>
-	<material name="LightGrey"/>
-    </visual>
-  </link>
-  <joint name="camera_top_link_joint" type="fixed">
-    <origin xyz="0.135 0 0.78"/>
-    <parent link="camera_base_link"/>
-    <child link="camera_top_link"/>
-  </joint>
-//////////////////////////////////////////////////////////////////////////////////////////////
-<link name="camera_link">
-    <visual>
-      <origin xyz="-0.055 0.0 -0.02 " />
-      <geometry>
-        <box size="0.11 0.03 0.04" />
-      </geometry>
-      <material name="test"/>
+        <visual>
+            <origin xyz="0.0 0.0 0.39"/>
+            <geometry>
+                <box size="0.03 0.03 0.78"/>
+            </geometry>
+            <material name="LightGrey"/>
+        </visual>
+    </link>
+    <joint name="camera_base_joint" type="fixed">
+        <origin xyz="-0.03 0.65 0.0"/>
+        <parent link="world"/>
+        <child link="camera_base_link"/>
+    </joint>
+    <link name="camera_top_link">
+        <visual>
+            <origin xyz="-0.25 0.0 0.015"/>
+            <geometry>
+                <box size="0.5 0.03 0.03"/>
+            </geometry>
+            <material name="LightGrey"/>
+        </visual>
+    </link>
+    <joint name="camera_top_link_joint" type="fixed">
+        <origin xyz="0.135 0 0.78"/>
+        <parent link="camera_base_link"/>
+        <child link="camera_top_link"/>
+    </joint>
+  <link name="camera_link">
+    <visual>
+      <origin xyz="-0.055 0.0 -0.2" />
+      <geometry>
+        <box size="0.0 0.0 0.0"/>
+      </geometry>
+      <material name="LightGrey"/>
     </visual>
   </link>
   <joint name="camera_joint" type="fixed">
-    <origin xyz="-0.39 0.0 0" />
-    <parent link="camera_top_link" />
+    <origin xyz="-0.305 0.64 0.76" rpy="1.53 1.53 3.1415" />
+    <parent link="world" />
     <child link="camera_link" />
   </joint>

Commit message: Add files via upload

File: src/my_xarm_lite6/urdf/lite6_robot.urdf.xacro (robot description, xacro)
@@ -204,5 +204,5 @@
   </link>
   <joint name="camera_joint" type="fixed">
-    <origin xyz="-0.305 0.64 0.76" rpy="1.53 1.53 3.1415" />
+    <origin xyz="-0.305 0.64 0.76" rpy="1.53 1.53 1.53" />
     <parent link="world" />
     <child link="camera_link" />
@@ -331,5 +331,5 @@
   </link>
  <joint name="Bak_drie" type="fixed">
-    <origin xyz="-0.105 -0.055 0.07" />
+    <origin xyz="-0.105 -0.110 0.07" />
     <parent link="Bak_een_link" />
     <child link="Bak_drie_link" />
@@ -373,5 +373,5 @@
   </link>
 <joint name="Bak_vier" type="fixed">
-    <origin xyz="0.0 -0.055 0.07" />
+    <origin xyz="0.0 -0.110 0.07" />
     <parent link="Bak_een_link" />
     <child link="Bak_vier_link" />

Commit message: Update lite6_robot.urdf.xacro
Nieuwe waardes Camera_Joint

File: src/my_xarm_lite6/urdf/lite6_robot.urdf.xacro (robot description, xacro)
@@ -204,5 +204,5 @@
   </link>
   <joint name="camera_joint" type="fixed">
-    <origin xyz="-0.305 0.64 0.76" rpy="1.53 1.53 1.53" />
+    <origin xyz="-0.235 0.61 0.76" rpy="1.53 1.53 1.53" />
     <parent link="world" />
     <child link="camera_link" />

Commit message: Update lite6_robot.urdf.xacro
wijziging camera_link

File: src/my_xarm_lite6/urdf/lite6_robot.urdf.xacro (robot description, xacro)
@@ -196,5 +196,5 @@
   <link name="camera_link">
     <visual>
-      <origin xyz="-0.055 0.0 -0.2" />
+      <origin xyz="0.0 0.0 0.0" />
       <geometry>
         <box size="0.0 0.0 0.0"/>
@@ -204,5 +204,5 @@
   </link>
   <joint name="camera_joint" type="fixed">
-    <origin xyz="-0.235 0.61 0.76" rpy="1.53 1.53 1.53" />
+    <origin xyz="-0.325 0.64 0.76" rpy="1.53 1.53 1.53" />
     <parent link="world" />
     <child link="camera_link" />

Commit message: Update lite6_robot.urdf.xacro
Wijziging camera_link

File: src/my_xarm_lite6/urdf/lite6_robot.urdf.xacro (robot description, xacro)
@@ -204,5 +204,5 @@
   </link>
   <joint name="camera_joint" type="fixed">
-    <origin xyz="-0.325 0.64 0.76" rpy="1.53 1.53 1.53" />
+    <origin xyz="-0.305 0.64 0.76" rpy="1.53 1.53 1.53" />
     <parent link="world" />
     <child link="camera_link" />

Commit message: Update lite6_robot.urdf.xacro
Toevoeging tandenborstel en wijziging camera

File: src/my_xarm_lite6/urdf/lite6_robot.urdf.xacro (robot description, xacro)
@@ -196,5 +196,5 @@
   <link name="camera_link">
     <visual>
-      <origin xyz="0.0 0.0 0.0" />
+      <origin xyz="-0.055 0.0 -0.2" />
       <geometry>
         <box size="0.0 0.0 0.0"/>
@@ -204,5 +204,5 @@
   </link>
   <joint name="camera_joint" type="fixed">
-    <origin xyz="-0.305 0.64 0.76" rpy="1.53 1.53 1.53" />
+    <origin xyz="-0.28 0.64 0.76" rpy="1.5708 1.5708 3.1415" />
     <parent link="world" />
     <child link="camera_link" />
@@ -394,7 +394,13 @@
     <visual>
       <geometry>
-        <box size="0.05 0.02 0.025" />
+        <box size="0.02 0.05 0.025" />
       </geometry>
       <material name="test"/>
+    </visual>
+    <visual>
+      <geometry>
+        <box size="0.19 0.02 0.02" />
+      </geometry>
+      <material name="blue"/>
     </visual>
   </link>

Commit message: los maken van borstel

File: src/my_xarm_lite6/urdf/lite6_robot.urdf.xacro (robot description, xacro)
@@ -398,4 +398,6 @@
       <material name="test"/>
     </visual>
+  </link>
+<link name="Borstel_link">
     <visual>
       <geometry>
@@ -405,4 +407,9 @@
     </visual>
   </link>
+<joint name="borstel" type="fixed">
+    <origin xyz="0.0 0.0 0.025" />
+    <parent link="cylinder_link" />
+    <child link="Borstel_link" />
+  </joint>
 <joint name="gripper" type="fixed">
     <origin xyz="0.0 0.0 0.025" />

Commit message: Update lite6_robot.urdf.xacro
Kleine wijziging locatie camera

File: src/my_xarm_lite6/urdf/lite6_robot.urdf.xacro (robot description, xacro)
@@ -204,5 +204,5 @@
   </link>
   <joint name="camera_joint" type="fixed">
-    <origin xyz="-0.28 0.64 0.76" rpy="1.5708 1.5708 3.1415" />
+    <origin xyz="-0.29 0.645 0.76" rpy="1.5708 1.5708 3.1415" />
     <parent link="world" />
     <child link="camera_link" />
@@ -398,6 +398,4 @@
       <material name="test"/>
     </visual>
-  </link>
-<link name="Borstel_link">
     <visual>
       <geometry>
@@ -407,9 +405,4 @@
     </visual>
   </link>
-<joint name="borstel" type="fixed">
-    <origin xyz="0.0 0.0 0.025" />
-    <parent link="cylinder_link" />
-    <child link="Borstel_link" />
-  </joint>
 <joint name="gripper" type="fixed">
     <origin xyz="0.0 0.0 0.025" />

Commit message: Update lite6_robot.urdf.xacro
toevoeging van muur

File: src/my_xarm_lite6/urdf/lite6_robot.urdf.xacro (robot description, xacro)
@@ -156,8 +156,21 @@
       <origin xyz="-0.15 0 0.1"/>
       <geometry>
-        <box size="0.30 0.06 0.22"/>
+        <box size="0.30 0.02 0.20"/>
       </geometry>
     </collision>
   </link>
+  <link name="muur_toren_link">
+    <collision>
+      <origin xyz="-0.15 0 0.1"/>
+      <geometry>
+        <box size="0.01 0.01 0.90"/>
+      </geometry>
+    </collision>
+  </link>
+  <joint name="muur_toren_joint" type="fixed">
+    <origin xyz="0.05 0.39 0" />
+    <parent link="world" />
+    <child link="muur_toren_link" />
+  </joint>
   <joint name="muur_joint" type="fixed">
     <origin xyz="-0.07 0.39 0" />
@@ -381,5 +394,5 @@
     <visual>
       <geometry>
-        <cylinder radius="0.0375" length="0.045"/>
+        <cylinder radius="0.0370" length="0.045"/>
       </geometry>
       <material name="test"/>
@@ -398,9 +411,11 @@
       <material name="test"/>
     </visual>
-    <visual>
-      <geometry>
-        <box size="0.19 0.02 0.02" />
-      </geometry>
-      <material name="blue"/>
+  </link>
+<link name="borstel_link">
+    <visual>
+      <geometry>
+        <box size="0.19 0.02 0.01" />
+      </geometry>
+      <material name="test"/>
     </visual>
   </link>
@@ -410,3 +425,8 @@
     <child link="gripper_link" />
   </joint>
+<joint name="borstel" type="fixed">
+    <origin xyz="0.0 0.0 0.04" />
+    <parent link="cylinder_link" />
+    <child link="borstel_link" />
+  </joint>
 </robot>

Commit message: Update lite6_robot.urdf.xacro
Toevoeging van vergroting Kabel Tool

File: src/my_xarm_lite6/urdf/lite6_robot.urdf.xacro (robot description, xacro)
@@ -420,4 +420,12 @@
     </visual>
   </link>
+<link name="kabel_link">
+    <visual>
+      <geometry>
+        <box size="0.01 0.06 0.015" />
+      </geometry>
+      <material name="test"/>
+    </visual>
+  </link>
 <joint name="gripper" type="fixed">
     <origin xyz="0.0 0.0 0.025" />
@@ -430,3 +438,8 @@
     <child link="borstel_link" />
   </joint>
+<joint name="kabel" type="fixed">
+    <origin xyz="0.0 0.04 -0.03" />
+    <parent link="cylinder_link" />
+    <child link="kabel_link" />
+  </joint>
 </robot>

Commit message: Update lite6_robot.urdf.xacro
Muur toren verwijderd

File: src/my_xarm_lite6/urdf/lite6_robot.urdf.xacro (robot description, xacro)
@@ -160,17 +160,4 @@
     </collision>
   </link>
-  <link name="muur_toren_link">
-    <collision>
-      <origin xyz="-0.15 0 0.1"/>
-      <geometry>
-        <box size="0.01 0.01 0.90"/>
-      </geometry>
-    </collision>
-  </link>
-  <joint name="muur_toren_joint" type="fixed">
-    <origin xyz="0.05 0.39 0" />
-    <parent link="world" />
-    <child link="muur_toren_link" />
-  </joint>
   <joint name="muur_joint" type="fixed">
     <origin xyz="-0.07 0.39 0" />

Commit message: Update lite6_robot.urdf.xacro

File: src/my_xarm_lite6/urdf/lite6_robot.urdf.xacro (robot description, xacro)
@@ -156,5 +156,5 @@
       <origin xyz="-0.15 0 0.1"/>
       <geometry>
-        <box size="0.30 0.02 0.20"/>
+        <box size="0.30 0.02 0.21"/>
       </geometry>
     </collision>
@@ -204,5 +204,5 @@
   </link>
   <joint name="camera_joint" type="fixed">
-    <origin xyz="-0.29 0.645 0.76" rpy="1.5708 1.5708 3.1415" />
+    <origin xyz="-0.30 0.64 0.74" rpy="1.5708 1.5708 3.1415" />
     <parent link="world" />
     <child link="camera_link" />
@@ -247,5 +247,5 @@
   </link>
   <joint name="Bak_een" type="fixed">
-    <origin xyz="-0.25 0.22 0.0" />
+    <origin xyz="-0.255 0.22 0.0" />
     <parent link="world" />
     <child link="Bak_een_link" />
@@ -289,5 +289,5 @@
   </link>
   <joint name="Bak_twee" type="fixed">
-    <origin xyz="-0.105 0.0 0.0" />
+    <origin xyz="-0.11 0.0 0.0" />
     <parent link="Bak_een_link" />
     <child link="Bak_twee_link" />
@@ -331,5 +331,5 @@
   </link>
  <joint name="Bak_drie" type="fixed">
-    <origin xyz="-0.105 -0.110 0.07" />
+    <origin xyz="-0.11 -0.110 0.07" />
     <parent link="Bak_een_link" />
     <child link="Bak_drie_link" />
@@ -381,5 +381,5 @@
     <visual>
       <geometry>
-        <cylinder radius="0.0370" length="0.045"/>
+        <cylinder radius="0.0370" length="0.050"/>
       </geometry>
       <material name="test"/>
@@ -394,5 +394,5 @@
     <visual>
       <geometry>
-        <box size="0.02 0.05 0.025" />
+        <box size="0.02 0.05 0.030" />
       </geometry>
       <material name="test"/>
